Commit message: 코드 정리.

File: models/pendulum.urdf (robot description, URDF)
Before this commit: robot pendulum, 4 links, 3 joints
Links:
- removed link ball
Joints:
- removed joint fixed_ball

Commit message: 클래스로 pybullet 환경 구성 완료.

File: models/pendulum.urdf (robot description, URDF)
Before this commit: robot pendulum, 3 links, 2 joints
Links:
- link base: mass 0.5 -> 1.0
